Commit message: added wrist joints back to the urdf model

File: models/valkyrie_simplified.urdf (robot description, URDF)
Before this commit: robot valkyrie, 84 links, 83 joints
Joints:
- joint leftWristPitch: type fixed -> revolute
- joint leftWristRoll: type fixed -> revolute
- joint rightWristPitch: type fixed -> revolute
- joint rightWristRoll: type fixed -> revolute

Commit message: modified valkyrie to remove collision meshes for large links. Updated the box to be a door like object

File: models/valkyrie_simplified.urdf (robot description, URDF)
Before this commit: robot valkyrie, 84 links, 83 joints
Links:
- link leftHipPitchLink: geometry collision cylinder length=0.35 radius=0.115; visual mesh filename=package://val_desc/model/meshes/legs/lj3_left.dae
- link leftShoulderRollLink: geometry collision cylinder length=0.176 radius=0.08; visual mesh filename=package://val_desc/model/meshes/arms/aj2_left.dae
- link rightHipPitchLink: geometry collision cylinder length=0.35 radius=0.115; visual mesh filename=package://val_desc/model/meshes/legs/lj3_right.dae
- link rightShoulderRollLink: geometry collision cylinder length=0.176 radius=0.08; visual mesh filename=package://val_desc/model/meshes/arms/aj2_right.dae
- link torso: geometry collision cylinder length=0.01 radius=0.2475; visual mesh filename=package://val_desc/model/meshes/torso/torso.dae
