Commit message: added new pseudo joint and object for the handle

File: models/test_cart.urdf (robot description, URDF)
Before this commit: robot cart, 1 links, 0 joints
Links:
- added link handle_link, mass 0.5; collision cylinder length=0.38 radius=0.0175; visual cylinder length=0.38 radius=0.0175
- link base_link: geometry collision box size=0.45 0.85 0.58; visual mesh filename=package://avatar_locomanipulation/models/cart/Trolley0.001.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
Joints:
- added joint handle_joint: type fixed, parent base_link, child handle_link, origin xyz=0.9335 0 0.9155 rpy=1.57 0 0, axis 1 0 0

Commit message: updates testing that the cart works, can be appended, etc

File: models/test_cart.urdf (robot description, URDF)
Before this commit: robot cart, 2 links, 1 joints
Joints:
- joint handle_joint: origin xyz=0.9335 0 0.9155 rpy=1.57 0 0 -> xyz=-0.5665 0 0.9155 rpy=1.57 0 0
