Commit message: fixed the collision for the head, which had been untouched

File: models/valkyrie_simplified_collisions.urdf (robot description, URDF)
Before this commit: robot valkyrie, 84 links, 83 joints
Links:
- link head: geometry collision box size=0.1311 0.12 0.15; collision sphere radius=0.0325
- link hokuyo_link: geometry visual mesh filename=package://val_desc/model/meshes/multisense/head_camera.dae

Commit message: 1)removed all environmental object functionality from collision environment due to the fact that it is wrong and will need to be rebuilt. 2) removed build_self_directed_vectors from collision environment to simplify testing. 3) currently build vectors to lhand and head are commented out, since i wanted a POC for correctly obtaining near_points. 4) commented out the computeError in task_selfcollision for testing purposes. 5) most of test_collision_environment commented out for testing and this will need to be rebuilt to reflect loss of functionality in collision env. 6) build_directed_vector_rhand works

File: models/valkyrie_simplified_collisions.urdf (robot description, URDF)
Before this commit: robot valkyrie, 84 links, 83 joints
Links:
- added link leftElbowNearLink, mass 0.0; collision sphere radius=0.085
- added link leftKneeNearLink, mass 0.0; collision sphere radius=0.095
- added link rightElbowNearLink, mass 0.0; collision sphere radius=0.085
- added link rightKneeNearLink, mass 0.0; collision sphere radius=0.095
Joints:
- added joint leftElbowNear: type fixed, parent leftShoulderYawLink, child leftElbowNearLink, origin xyz=0.0254 0.33 0.0 rpy=0.0 0.0 0.0, axis 0 0 1
- added joint leftKneeNear: type fixed, parent leftHipPitchLink, child leftKneeNearLink, origin xyz=0.000112225 0.0361046 -0.430959 rpy=0.0 0.0 0.0, axis 0 1 0
- added joint rightElbowNear: type fixed, parent rightShoulderYawLink, child rightElbowNearLink, origin xyz=0.0254 -0.33 0.0 rpy=0.0 0.0 0.0, axis 0 0 1
- added joint rightKneeNear: type fixed, parent rightHipPitchLink, child rightKneeNearLink, origin xyz=0.000112225 -0.0361046 -0.430959 rpy=0.0 0.0 0.0, axis 0 1 0

Commit message: added some notes to collision env. added a new task checking multiple self collision tasks. added build_directed_vectors_to_wrists and included those in the selfcollision task. changed the Potential in get_collision_dx

File: models/valkyrie_simplified_collisions.urdf (robot description, URDF)
Before this commit: robot valkyrie, 88 links, 87 joints
Links:
- link pelvis: geometry collision box size=0.2 0.25 0.25; visual mesh filename=package://val_desc/model/meshes/pelvis/pelvis.dae

Commit message: fixed the issues with self collision avoidance merely causing other self collisions. Added a flag to directed vectors indicating if the links are in collision- >using this to change the safety_distance. Changed the urdf to treat hip upper and hip lower as diff links and changed collision env accordingly

File: models/valkyrie_simplified_collisions.urdf (robot description, URDF)
Before this commit: robot valkyrie, 88 links, 87 joints
Links:
- added link leftHipUpperLink, mass 10.2; collision box size=0.125 0.065 0.19
- added link rightHipUpperLink, mass 10.2; collision box size=0.125 0.065 0.19
- link leftHipPitchLink: geometry collision cylinder length=0.25 radius=0.075; visual mesh filename=package://val_desc/model/meshes/legs/lj3_left.dae
- link rightHipPitchLink: geometry collision cylinder length=0.25 radius=0.075; visual mesh filename=package://val_desc/model/meshes/legs/lj3_right.dae
Joints:
- added joint leftHipUpper: type fixed, parent leftHipPitchLink, child leftHipUpperLink, origin xyz=0.0 0.0 -0.0609 rpy=0.0 0.0 0.0, axis 0 1 0, limit lower=-2.42 upper=1.619 effort=350 velocity=6.11
- added joint rightHipUpper: type fixed, parent rightHipPitchLink, child rightHipUpperLink, origin xyz=0.0 0.0 -0.0609 rpy=0.0 0.0 0.0, axis 0 1 0, limit lower=-2.42 upper=1.619 effort=350 velocity=6.11
