Commit message: removed some previous debugging from collision env. changed the two boxes to be 2 and 1 cm instead of 10 and 20. added box visualization to the multiple object test file. Tested to see that the robot does avoid the objects in two cases: 1) objects near both hands, 2) objects near only one hand. It works in both cases, though error is never driven to 0. The task gains were set to 1 and the pelvis position task was removed

File: models/simplebox1.urdf (robot description, URDF)
Before this commit: robot box20, 1 links, 0 joints
Links:
- removed link box20
- added link box1, mass 3.0; collision box size=0.01 0.01 0.01; visual box size=0.01 0.01 0.01

File: models/simplebox2.urdf (robot description, URDF)
Before this commit: robot box10, 1 links, 0 joints
Links:
- removed link box10
- added link box2, mass 3.0; collision box size=0.02 0.02 0.02; visual box size=0.02 0.02 0.02
