Commit message: free ankle limits

File: models/valkyrie_no_fingers.urdf (robot description, URDF)
Before this commit: robot valkyrie, 42 links, 41 joints
Joints:
- joint leftAnklePitch: limit lower=-0.8644 upper=0.875 effort=205 velocity=11 -> lower=-1.8644 upper=1.875 effort=205 velocity=11
- joint leftAnkleRoll: limit lower=-0.349 upper=0.348 effort=205 velocity=11 -> lower=-1.349 upper=1.348 effort=205 velocity=11
- joint rightAnklePitch: limit lower=-0.8644 upper=0.875 effort=205 velocity=11 -> lower=-1.8644 upper=1.875 effort=205 velocity=11
- joint rightAnkleRoll: limit lower=-0.349 upper=0.348 effort=205 velocity=11 -> lower=-1.349 upper=1.348 effort=205 velocity=11

Commit message: 0.56 trajectory. free up wrist limits. torso posture task change, but no obvious impact.

File: models/valkyrie_no_fingers.urdf (robot description, URDF)
Before this commit: robot valkyrie, 42 links, 41 joints
Joints:
- joint rightWristPitch: limit lower=-0.49 upper=0.36 effort=14 velocity=1 -> lower=-3.14 upper=3.14 effort=14 velocity=1
- joint rightWristRoll: limit lower=-0.625 upper=0.62 effort=14 velocity=1 -> lower=-3.14 upper=3.14 effort=14 velocity=1

Commit message: 9 sec. result for nn

File: models/valkyrie_no_fingers.urdf (robot description, URDF)
Before this commit: robot valkyrie, 42 links, 41 joints
Joints:
- joint leftWristPitch: limit lower=-0.36 upper=0.49 effort=14 velocity=1 -> lower=-3.14 upper=3.14 effort=14 velocity=1
- joint leftWristRoll: limit lower=-0.62 upper=0.625 effort=14 velocity=1 -> lower=-3.14 upper=3.14 effort=14 velocity=1

Commit message: pushing to 0.32

File: models/valkyrie_no_fingers.urdf (robot description, URDF)
Before this commit: robot valkyrie, 42 links, 41 joints
Joints:
- joint rightWristPitch: limit lower=-3.14 upper=3.14 effort=14 velocity=1 -> lower=-4.14 upper=4.14 effort=14 velocity=1
- joint rightWristRoll: limit lower=-3.14 upper=3.14 effort=14 velocity=1 -> lower=-4.14 upper=4.14 effort=14 velocity=1

Commit message: renamed files. added dedicated isualization scripts. visualize once enabled for just the configuration

File: models/valkyrie_no_fingers.urdf (robot description, URDF)
Before this commit: robot valkyrie, 42 links, 41 joints
Joints:
- joint rightWristPitch: limit lower=-4.14 upper=4.14 effort=14 velocity=1 -> lower=-3.14 upper=3.14 effort=14 velocity=1
- joint rightWristRoll: limit lower=-4.14 upper=4.14 effort=14 velocity=1 -> lower=-3.14 upper=3.14 effort=14 velocity=1
